File: hw/Drivers.sch (KiCad schematic (older format))
At the start: 56 parts, among them Q1 ZVP2110A, Q10 2N3904, Q11 2N3904, Q12 2N3904, Q13 2N3904, Q14 2N3904, Q15 2N3904, Q16 2N3904, Q17 2N3904, Q18 2N3904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

Commit message: Initial PCB part layout
Still no keyboard or audio out, but I have ideas for those that
shouldn't cause too much havoc with my schematic.  I hope.
Parts:
- removed Q10, Q11, Q12, Q13, Q14, Q15, Q16, Q17, Q18, Q19, Q20, Q21, Q22, Q23, Q24, Q25, Q26, Q27, Q28, Q9: 2N3904, symbol NPN
- added Q10, Q11, Q12, Q13, Q14, Q15, Q16, Q17, Q18, Q19, Q20, Q21, Q22, Q23, Q24, Q25, Q26, Q27, Q28, Q9: 2N3904, TO92-EBC, symbol BC237
