File: hw/SpaceTime.sch (KiCad schematic (older format))
At the start: 47 parts, among them J1 JACK_2P, P1 AVR-ISP-6, P2 CONN_6, P3 Current time, P4 Open till, P5 Cleanup time, SW1 SW_PUSH, U1 ATMEGA328P-P, U2 74HC595, U3 74HC595, U4 74HC595, U5 L7812ABV, U6 LM1086

Commit message: Added bypass caps on shift registers (optional, but easier to add now) Messed with junctions that were needed for ERC to pass (on recent Mac build, but not on older Windows build)
Parts:
- added C10, C11, C12: 0.1uF, symbol C
Connections:
- net labels added: 5V-A, 5V-B, 5V-C
- wire segments 131 -> 140

Commit message: Changed connectors to style I could get locally Swapped on-board 12v regulation for external 12v regulated supply
Parts:
- removed C8, C9: 10uF, symbol C
- removed P3: Current time, symbol CONN_12
- removed P4: Open till, symbol CONN_12
- removed P5: Cleanup time, symbol CONN_12
- removed U5: L7812ABV, symbol L7812ABV
- added D2: Power, symbol LED
- added IID-J1, IID-J2, IID-J3, IID-P1, IID-P10, IID-P11, IID-P12, IID-P2, IID-P3, IID-P4, IID-P5, IID-P6, IID-P7, IID-P8, IID-P9: CONN_1, symbol CONN_1
- added P3: Current time, symbol CONN_8X2
- added P4: Open till, symbol CONN_8X2
- added P5: Cleanup time, symbol CONN_8X2
- added R30: 150, symbol R
- P1: value AVR-ISP-6 -> AVR-ISP
- P2: value CONN_6 -> Serial
- SW1: value SW_PUSH -> Reset
- renumbered U1 to MCU1, U6 to U1
Connections:
- wire segments 140 -> 143
Other:
- note removed: "(14-24VDC)"
- moved on the sheet: C4, C5, C6, C7, D1, J1, U1, XTL1

Commit message: Updated Readme with more detail of what I'm up to Renamed one connector on the main board
Parts:
- P4: value Open till -> Closing time
Changed lines of the file:
@@
-EESchema Schematic File Version 2  date Wednesday, 13 February, 2013 08:52:21 pm
+EESchema Schematic File Version 2  date Wednesday, 13 February, 2013 08:58:23 pm
 LIBS:SpaceTime
 LIBS:power
@@
 P 10050 2700
 F 0 "P4" H 10050 3150 60  0000 C CNN
-F 1 "Open till" V 10050 2700 50  0000 C CNN
+F 1 "Closing time" V 10050 2700 50  0000 C CNN
 	1    10050 2700
 	1    0    0    -1

Commit message: Initial PCB part layout
Still no keyboard or audio out, but I have ideas for those that
shouldn't cause too much havoc with my schematic.  I hope.
Parts:
- removed C6, C7: 10uF, symbol C
- added C6, C7: 10uF, symbol CP1
- added IID-G1, IID-V1: CONN_1, symbol CONN_1
- added R31, R32, R33: 10k, symbol R
Other:
- moved on the sheet: IID-J1, IID-J2, IID-J3, IID-S4, IID-S5, IID-S6, IID-S7, J1

Commit message: Partially routed PCB
Should be able to tighten up the board outline a bit from here, we'll
see.
Parts:
- removed IID-26, IID-27, IID-28, IID-4, IID-5, IID-S4, IID-S5, IID-S6, IID-S7: CONN_1, symbol CONN_1
- added P6: SPK, symbol CONN_2
- added P7: Keyboard, symbol CONN_8
- added Q29: ZVP2110A, symbol MOSFET_P
- added Q30: 2N3904, TO92-EBC, symbol BC237
- added R34: 40k, symbol R
- added R35: 1k, symbol R
Connections:
- net labels added: KI-1, KI-2, KI-3, KI-4, KO-1, KO-2, KO-3, KO-4, Spk
- wire segments 143 -> 150

Commit message: PCB is starting to shape up
Need to sort out PWM for shift registers, then some power and ground.
Parts:
- added D3, D4, D5: DIODE, symbol DIODE
- added M1, M2, M3, M4: MOUNTING_HOLE, symbol MOUNTING_HOLE
- added RX1, Skip1, Skip2, TX1: CONN_1, symbol CONN_1
- renumbered IID-11 to A11, IID-12 to A12, IID-13 to A13, IID-14 to A14, IID-6 to A6, IID-21 to Aref1, IID-P1 to Extra1, IID-P10 to Extra10, IID-P11 to Extra11, IID-P12 to Extra12, IID-P2 to Extra2, IID-P3 to Extra3, IID-P4 to Extra4, IID-P5 to Extra5, IID-P6 to Extra6, IID-P7 to Extra7, IID-P8 to Extra8, IID-P9 to Extra9, IID-G1 to G1, IID-J1 to Ja1, IID-J2 to Ja2, IID-J3 to Ja3, IID-SER1 to SER1, IID-SER2 to SER2, IID-SER3 to SER3, IID-SER4 to SER4, IID-SER5 to SER5, IID-SER6 to SER6, IID-S9 to Sout-1, IID-V1 to V1
Connections:
- wire segments 150 -> 152
Other:
- moved on the sheet: C6, C7, D1, D2, G1, P2, P7, R30, SER1, SER2, SER3, SER4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

Commit message: PCB passes DRC!
Need to nail down pad on 5V regulator, if nothing else.
Parts:
- removed A11, A12: CONN_1, symbol CONN_1
- added A23: CONN_1, symbol CONN_1
Connections:
- wire segments 152 -> 153
Other:
- moved on the sheet: R31, R33
