File: hw/SpaceTime.sch (KiCad schematic (older format))
At the start: 76 parts, among them J1 JACK_2P, M1 MOUNTING_HOLE, M2 MOUNTING_HOLE, M3 MOUNTING_HOLE, M4 MOUNTING_HOLE, P1 AVR-ISP, P2 Serial, P3 Current time, P4 Closing time, P5 Cleanup time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

Commit message: Shrunk board, went with SMT driver section
Lots of changes...
Shrank board to fit ITEAD Studio 10x10cm board size
Dropped 3rd shirt register, use segment scan for keyboard
Switched repetitive driver sections to SMT parts
Parts:
- removed A23, Extra10, Extra11, Extra12, Extra9, Skip1, Skip2: CONN_1, symbol CONN_1
- removed C12: 0.1uF, symbol C
- removed D3, D4, D5: DIODE, symbol DIODE
- removed P5: Cleanup time, symbol CONN_8X2
- removed R33: 10k, symbol R
- removed U4: 74HC595, symbol 74HC595
- added A11, A12, A5: CONN_1, symbol CONN_1
- Q29: value ZVP2110A -> BSH202,215
- Q30: value 2N3904 -> MMBT3904
Connections:
- net labels removed: 5V-C, CC 3:1, CC 3:2, CC 3:3, CC 3:4
- wire segments 153 -> 131
Other:
- moved on the sheet: C6, C7, D1, D2, G1, Ja1, Ja2, Ja3, P2, R30, R31, R32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

Commit message: Board design completed (I hope)
This is the 1.0 version of the board, as mailed off for PCB
manufacturing.
Parts:
- removed U1: LM1086, symbol LM1086
- added C12: 0.1uF, symbol C
- added U1: LM7805, symbol LM7805
Connections:
- wire segments 131 -> 133
Other:
- moved on the sheet: C7, D2, R30
